File: electronics/esp8266-nrf51-configurator/esp8266-nrf51-configurator.sch (KiCad schematic (older format))
At the start: 9 parts, among them K1 ESP-PROG, P1 LOG, P2 nRF-UART, P3 SWD, SW1 On/Off, U1 ESP8266_R2, U2 LIPO_CHARGER_+_PROTECTION, U3 CORE51822B

Commit message: Update schematics
Other:
- note added: "Tapped off the 3.3V regulator\non the ESP8266 R2 PCB"
- note removed: "From 3.3V regulator\non the ESP8266 R2 PCB"
Changed lines of the file:
@@
 LIBS:contrib
 LIBS:valves
+LIBS:esp8266-nrf51-configurator-cache
 EELAYER 27 0
 EELAYER END
@@
 	3900 3200 5100 3200
 Text Notes 3350 2050 0    60   ~ 0
-From 3.3V regulator\non the ESP8266 R2 PCB
+Tapped off the  3.3V regulator\non the ESP8266 R2 PCB
 Text Notes 5200 3600 0    60   ~ 0
 Debug log messages\nUART 115200
