File: configurator/usb-dongle/electronics/usb-dongle.kicad_pcb (KiCad board)
At the start: 2 copper layers, 29 parts, among them K1 CONN_3, K10 CONN_3, K11 CONN_3, K2 CONN_3, K3 CONN_3, K4 CONN_3, K5 CONN_3, K6 CONN_3, K7 CONN_3, K8 CONN_3, K9 CONN_3, P1 Charge, P2 LED, P3 CONN_2, P4 CONN_2, P5 CONN_4, Q1 BC548, SW1 ON/OFF, U1 LIPO_CHARGER_+_PROTECTION, U2 STM32F103C8T6_DEV_BOARD, U3 NRF24L01P

Commit message: Kicad 5 version and schematic update
Parts:
- removed BT1: BATTERY, PIN_ARRAY_2X1
- removed C1: 1u, SM0805
- removed C2: 100nF, SM0805
- removed K1, K10, K11, K2, K3, K4, K5, K6, K7, K8, K9: CONN_3, PIN_ARRAY_3X1
- removed P1: Charge, PIN_ARRAY_2X1
- removed P2: LED, PIN_ARRAY_2X1
- removed P3, P4: CONN_2, PIN_ARRAY_2X1
- removed P5: CONN_4, PIN_ARRAY_4x1
- removed Q1: BC548, TO92
- removed R1, R4: 1k, SM0805
- removed R2, R3: R, SM0805
- removed SP1: SPEAKER, PIN_ARRAY_2X1
- removed SW1: ON/OFF, PIN_ARRAY_2X1
- removed U1: LIPO_CHARGER_+_PROTECTION, LiPo_charger_and_protection
- removed U3: NRF24L01P, NRF24L01P-PA-LNA
Connections:
- U2 pad 1: /CSN -> (no net)
- U2 pad 10: /BUZZER -> (no net)
- U2 pad 18: VDD -> (no net)
- U2 pad 2: /SCK -> (no net)
- U2 pad 20: N-0000022 -> VCC
- U2 pad 21: N-0000022 -> VCC
- U2 pad 22: /LED -> (no net)
- U2 pad 25: /ADC0 -> (no net)
- U2 pad 26: /ADC1 -> (no net)
- U2 pad 27: /ADC2 -> (no net)
- U2 pad 28: /ADC3 -> (no net)
- U2 pad 29: /ADC4 -> (no net)
- U2 pad 3: /MISO -> (no net)
- U2 pad 30: /ADC5 -> (no net)
- U2 pad 31: /ADC6 -> (no net)
- U2 pad 32: /ADC7 -> (no net)
- U2 pad 33: /ADC8 -> (no net)
- U2 pad 34: /ADC9 -> (no net)
- U2 pad 35: /SW2 -> (no net)
- U2 pad 36: /SW1 -> (no net)
- U2 pad 38: VCC -> (no net)
- U2 pad 4: /MOSI -> (no net)
- U2 pad 5: /IRQ -> (no net)
- U2 pad 6: /TX -> (no net)
- U2 pad 7: /RX -> (no net)
Routing:
- net VCC: track 122.5 -> 0.00 mm, vias 2 -> 0
- net GND: track 122.4 -> 0.00 mm, vias 4 -> 0
- net /SCK: track 33.0 -> 0.00 mm, vias 2 -> 0
- net /MISO: track 27.9 -> 0.00 mm, vias 2 -> 0
- net /IRQ: track 25.4 -> 0.00 mm
- net /ADC0: track 20.5 -> 0.00 mm
- net /MOSI: track 20.3 -> 0.00 mm
- net N-0000022: track 15.2 -> 0.00 mm
- net N-0000014: track 15.2 -> 0.00 mm
- net VDD: track 12.4 -> 0.00 mm
- net /CSN: track 10.2 -> 0.00 mm
- net N-0000029: track 8.45 -> 0.00 mm
- net N-000004: track 7.82 -> 0.00 mm
- net N-0000021: track 7.82 -> 0.00 mm
- net N-0000028: track 6.61 -> 0.00 mm
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Other:
- board text removed: "IMPORTANT: the nRF module is on the back side, i.e mirrored!"
