File: configurator/usb-dongle/electronics/usb-dongle.sch (KiCad schematic (older format))
At the start: 3 parts, among them U2 STM32F103C8T6_DEV_BOARD, U3 NRF24L01P

Commit message: Kicad 5 version and schematic update
Parts:
- removed C1: 1u, Capacitors_SMD:C_0805_HandSoldering, symbol C
- removed U3: NRF24L01P, WLA:NRF24L01P-PA-LNA, symbol NRF24L01P
- added U1: NRF51822_MODULE, symbol WLA-nrf51822-module:NRF51822_MODULE
- U2: symbol STM32F103C8T6_DEV_BOARD -> WLA-STM32:STM32F103C8T6_DEV_BOARD
Connections:
- net labels added: NRF_RX, NRF_TX, SWCLK, SWDIO, TX_PRINTF
- net labels removed: ADC0, BUZZER, CE, CSN, IRQ, LED, MISO, MOSI, PA1/ADC1, PA2/ADC2, PA3/ADC3, PA4/ADC4, PA5/ADC5, PA6/ADC6, PA7/ADC7, PB0/ADC8, PB1/ADC9, PB10, PB11, PB3, PB4, PB5, PB6, PB7, PB8, PB9, RX, SCK, TX, VDD
- wire segments 49 -> 19
- no-connect marks 11 -> 62
Other:
- note added: "Debug info 15200/N/8/1"
- moved on the sheet: U2
