File: transmitter/electronics/airtronics/stm32f1-nrf24l01-transmitter-airtronics.sch (KiCad schematic (older format))
At the start: 34 parts, among them K1 CONN_3, K10 CONN_3, K11 CONN_3, K12 UART, K2 CONN_3, K3 CONN_3, K4 CONN_3, K5 CONN_3, K6 CONN_3, K7 CONN_3, K8 CONN_3, K9 CONN_3, P1 Charge, P2 LED, P3 PWR-BAT, P4 PWR-IN, P5 Buzzer, P6 Meter, Q1 BC547B, SW1 ON/OFF, U1 LIPO_CHARGER_+_PROTECTION, U2 STM32F103C8T6_DEV_BOARD, U3 NRF24L01P

Commit message: Clean up electronics for latest KiCad
Parts:
- BT1: symbol BATTERY -> stm32f1-nrf24l01-transmitter-rescue:BATTERY
- C1, C2: symbol C-RESCUE-stm32f1-nrf24l01-transmitter -> stm32f1-nrf24l01-transmitter-rescue:C-RESCUE-stm32f1-nrf24l01-transmitter
- C3, C4: symbol C -> stm32f1-nrf24l01-transmitter-rescue:C
- K1, K10, K11, K12, K2, K3, K4, K5, K6, K7, K8, K9: symbol CONN_3 -> stm32f1-nrf24l01-transmitter-rescue:CONN_3
- P1, P2, P3, P4, P5, P6: symbol CONN_2 -> stm32f1-nrf24l01-transmitter-rescue:CONN_2
- Q1: symbol Q_NPN_CBE -> stm32f1-nrf24l01-transmitter-rescue:Q_NPN_CBE
- R1, R2, R3, R4, R5: symbol R-RESCUE-stm32f1-nrf24l01-transmitter -> stm32f1-nrf24l01-transmitter-rescue:R-RESCUE-stm32f1-nrf24l01-transmitter
- SP1: symbol SPEAKER -> stm32f1-nrf24l01-transmitter-rescue:SPEAKER
- SW1: symbol SPST -> stm32f1-nrf24l01-transmitter-rescue:SPST
- U1: symbol LIPO_CHARGER_+_PROTECTION -> stm32f1-nrf24l01-transmitter-rescue:LIPO_CHARGER_+_PROTECTION
- U2: symbol STM32F103C8T6_DEV_BOARD -> stm32f1-nrf24l01-transmitter-rescue:STM32F103C8T6_DEV_BOARD
- U3: symbol NRF24L01P -> stm32f1-nrf24l01-transmitter-rescue:NRF24L01P
