File: transmitter/electronics/pcb/stm32f1-nrf24l01-transmitter-pcb.sch (KiCad schematic (older format))
At the start: 69 parts, among them J1 PA1/A1, J10 PB3, J11 PB4, J12 PB5, J13 PB6, J14 PB7, J15 PB8, J16 PB10, J17 PB11, J18 External charger LED, J19 BATTERY, J2 PA2/A2, J20 Red, J21 Blue, J22 POWER SWITCH, J23 USB, J24 UART, J25 SWD, J26 Buzzer, J27 NRF24 connector, J28 NRF24 module, J29 Meter, J3 PA3/A3, J30 LED, J4 PA4/A4, J5 PA5/A5, J6 PA6/A6, J7 PA7/A7, J8 PB0/A8, J9 PB1/A9, Q1 PMV30UN, SW1 RESET, U1 MCP1703A-3302, U2 LIPO_CHARGER_+_PROTECTION, U3 STM32F103CBT6, U4 MCP1703A-3302, Y1 8MHz

Commit message: Work on schematics and layout
Parts:
- removed J28: NRF24 module, Connector_PinHeader_2.54mm:PinHeader_1x04_P2.54mm_Vertical, symbol Connector_Generic:Conn_01x04
- J25: footprint Connector_PinHeader_2.54mm:PinHeader_1x04_P2.54mm_Vertical -> Connector_PinHeader_2.54mm:PinHeader_1x03_P2.54mm_Vertical; symbol Connector_Generic:Conn_01x04 -> Connector_Generic:Conn_01x03
- SP1: footprint Buzzer_Beeper:Buzzer_12x9.5RM7.6 -> Buzzer_Beeper:MagneticBuzzer_PUI_AT-0927-TT-6-R
Connections:
- net +3V3: no longer J25.4 (Pin_4)
- net CE renamed 3V3_RF
Other:
- note removed: "Note that 4 pins of J22 and J? are \nmade to overlap, so that we can either\nmount a JST XH connector for wires to\nan external module, or a pin header for \ndirect NRF module mounting."
Changed lines of the file:
@@
 F 0 "SP1" H 14500 4600 70  0000 C CNN
 F 1 "SPEAKER" H 14500 4100 70  0001 C CNN
-F 2 "Buzzer_Beeper:Buzzer_12x9.5RM7.6" H 14600 4350 60  0001 C CNN
+F 2 "Buzzer_Beeper:MagneticBuzzer_PUI_AT-0927-TT-6-R" H 14600 4350 60  0001 C CNN
 F 3 "~" H 14600 4350 60  0000 C CNN
 	1    14600 4350
@@
 $EndComp
 Wire Wire Line
-	13150 2350 13150 2650
-Wire Wire Line
 	13600 2250 13900 2250
 Wire Wire Line
@@
 Wire Wire Line
 	13000 1950 13900 1950
-Wire Wire Line
-	13000 1850 13300 1850
 Text Label 13000 2150 0    50   ~ 0
 CSN
@@
 Wire Wire Line
 	5350 8750 5650 8750
-Text Notes 14250 2350 0    50   ~ 0
-Note that 4 pins of J22 and J? are \nmade to overlap, so that we can either\nmount a JST XH connector for wires to\nan external module, or a pin header for \ndirect NRF module mounting.
 $Comp
 L Mechanical:MountingHole H1
@@
 Wire Wire Line
 	12800 4850 13450 4850
-$Comp
-L Connector_Generic:Conn_01x04 J28
-U 1 1 5EF456C6
-P 14100 2750
-F 0 "J28" H 14180 2742 50  0000 L CNN
-F 1 "NRF24 module" H 14180 2651 50  0000 L CNN
-F 2 "Connector_PinHeader_2.54mm:PinHeader_1x04_P2.54mm_Vertical" H 14100 2750 50  0001 C CNN
-F 3 "~" H 14100 2750 50  0001 C CNN
-	1    14100 2750
-	1    0    0    -1
-$EndComp
-Text Label 13800 2750 0    50   ~ 0
-CE
-Wire Wire Line
-	13450 2850 13900 2850
 Wire Wire Line
 	12150 1300 12600 1300
@@
 	13600 1300 13600 2250
 Wire Wire Line
-	13000 1750 13450 1750
-Connection ~ 13450 1750
-Wire Wire Line
-	13450 1750 13900 1750
-Wire Wire Line
-	13450 1750 13450 2850
-Wire Wire Line
-	13300 2950 13300 1850
-Wire Wire Line
-	13300 2950 13900 2950
-Connection ~ 13300 1850
-Wire Wire Line
-	13300 1850 13900 1850
-Wire Wire Line
-	13600 2250 13600 2750
-Wire Wire Line
-	13600 2750 13900 2750
-Connection ~ 13600 2250
-Wire Wire Line
-	13150 2350 13900 2350
-Wire Wire Line
-	13150 2650 13900 2650
-Connection ~ 13150 2650
-Wire Wire Line
-	13150 2650 13150 3000
+	13600 2350 13900 2350
 Text Notes 12650 1000 0    79   ~ 16
 NRF24L01-PA-LNA module
@@
 L power:GND #PWR034
 U 1 1 5F2A3EFA
-P 13150 3000
-F 0 "#PWR034" H 13150 2750 50  0001 C CNN
-F 1 "GND" H 13155 2827 50  0000 C CNN
-F 2 "" H 13150 3000 50  0001 C CNN
-F 3 "" H 13150 3000 50  0001 C CNN
-	1    13150 3000
+P 13600 3000
+F 0 "#PWR034" H 13600 2750 50  0001 C CNN
+F 1 "GND" H 13605 2827 50  0000 C CNN
+F 2 "" H 13600 3000 50  0001 C CNN
+F 3 "" H 13600 3000 50  0001 C CNN
+	1    13600 3000
 	1    0    0    -1
 $EndComp
@@
 RESET
 $Comp
-L Connector_Generic:Conn_01x04 J25
+L Connector_Generic:Conn_01x03 J25
 U 1 1 5FABE4DE
 P 12400 9050
-F 0 "J25" H 12318 8625 50  0000 C CNN
-F 1 "SWD" H 12318 8716 50  0000 C CNN
-F 2 "Connector_PinHeader_2.54mm:PinHeader_1x04_P2.54mm_Vertical" H 12400 9050 50  0001 C CNN
+F 0 "J25" H 12400 8700 50  0000 C CNN
+F 1 "SWD" H 12400 8800 50  0000 C CNN
+F 2 "Connector_PinHeader_2.54mm:PinHeader_1x03_P2.54mm_Vertical" H 12400 9050 50  0001 C CNN
 F 3 "~" H 12400 9050 50  0001 C CNN
 	1    12400 9050
@@
 Wire Wire Line
 	11550 8950 12200 8950
-$Comp
-L power:+3V3 #PWR030
-U 1 1 5FB26DF6
-P 12100 8600
-F 0 "#PWR030" H 12100 8450 50  0001 C CNN
-F 1 "+3V3" H 12115 8773 50  0000 C CNN
-F 2 "" H 12100 8600 50  0001 C CNN
-F 3 "" H 12100 8600 50  0001 C CNN
-	1    12100 8600
-	1    0    0    -1
-$EndComp
-Wire Wire Line
-	12200 8850 12100 8850
-Wire Wire Line
-	12100 8850 12100 8600
 Text Label 11550 8950 0    50   ~ 0
 SWDIO
@@
 	1    0    0    1
 $EndComp
+Wire Wire Line
+	13600 2350 13600 3000
+Wire Wire Line
+	13000 1750 13900 1750
+Wire Wire Line
+	13000 1850 13900 1850
+Text Label 13200 1300 0    50   ~ 0
+3V3_RF
 $EndSCHEMATC

Commit message: Work on layout
Parts:
- added H3: MountingHole, MountingHole:MountingHole_3.2mm_M3_DIN965, symbol Mechanical:MountingHole
- Q1, U1, U4: footprint Package_TO_SOT_SMD:SOT-23 -> Package_TO_SOT_SMD:SOT-23_Handsoldering
Other:
- moved on the sheet: H1, H2
Changed lines of the file:
@@
 L Mechanical:MountingHole H1
 U 1 1 5E38CF71
-P 10950 10700
-F 0 "H1" H 11050 10746 50  0000 L CNN
-F 1 "MountingHole" H 11050 10655 50  0000 L CNN
-F 2 "MountingHole:MountingHole_3.2mm_M3_DIN965" H 10950 10700 50  0001 C CNN
-F 3 "~" H 10950 10700 50  0001 C CNN
-	1    10950 10700
+P 11000 10350
+F 0 "H1" H 11100 10396 50  0000 L CNN
+F 1 "MountingHole" H 11100 10305 50  0000 L CNN
+F 2 "MountingHole:MountingHole_3.2mm_M3_DIN965" H 11000 10350 50  0001 C CNN
+F 3 "~" H 11000 10350 50  0001 C CNN
+	1    11000 10350
 	1    0    0    -1
 $EndComp
@@
 L Mechanical:MountingHole H2
 U 1 1 5E38F132
-P 10950 10950
-F 0 "H2" H 11050 10996 50  0000 L CNN
-F 1 "MountingHole" H 11050 10905 50  0000 L CNN
-F 2 "MountingHole:MountingHole_3.2mm_M3_DIN965" H 10950 10950 50  0001 C CNN
-F 3 "~" H 10950 10950 50  0001 C CNN
-	1    10950 10950
+P 11000 10600
+F 0 "H2" H 11100 10646 50  0000 L CNN
+F 1 "MountingHole" H 11100 10555 50  0000 L CNN
+F 2 "MountingHole:MountingHole_3.2mm_M3_DIN965" H 11000 10600 50  0001 C CNN
+F 3 "~" H 11000 10600 50  0001 C CNN
+	1    11000 10600
 	1    0    0    -1
 $EndComp
@@
 F 0 "Q1" H 13854 4896 50  0000 L CNN
 F 1 "PMV30UN" H 13854 4805 50  0000 L CNN
-F 2 "Package_TO_SOT_SMD:SOT-23" H 13850 4775 50  0001 L CIN
+F 2 "Package_TO_SOT_SMD:SOT-23_Handsoldering" H 13850 4775 50  0001 L CIN
 F 3 "https://www.fairchildsemi.com/datasheets/BS/BSS138.pdf" H 13650 4850 50  0001 L CNN
 	1    13650 4850
@@
 F 0 "U4" H 11650 1542 50  0000 C CNN
 F 1 "MCP1703A-3302" H 11650 1451 50  0000 C CNN
-F 2 "Package_TO_SOT_SMD:SOT-23" H 11650 1500 50  0001 C CNN
+F 2 "Package_TO_SOT_SMD:SOT-23_Handsoldering" H 11650 1500 50  0001 C CNN
 F 3 "http://ww1.microchip.com/downloads/en/DeviceDoc/20005122B.pdf" H 11650 1250 50  0001 C CNN
 	1    11650 1300
@@
 F 0 "U1" H 4800 6392 50  0000 C CNN
 F 1 "MCP1703A-3302" H 4800 6301 50  0000 C CNN
-F 2 "Package_TO_SOT_SMD:SOT-23" H 4800 6350 50  0001 C CNN
+F 2 "Package_TO_SOT_SMD:SOT-23_Handsoldering" H 4800 6350 50  0001 C CNN
 F 3 "http://ww1.microchip.com/downloads/en/DeviceDoc/20005122B.pdf" H 4800 6100 50  0001 C CNN
 	1    4800 6150
@@
 Text Label 13200 1300 0    50   ~ 0
 3V3_RF
+$Comp
+L Mechanical:MountingHole H3
+U 1 1 5E292C58
+P 11000 10850
+F 0 "H3" H 11100 10896 50  0000 L CNN
+F 1 "MountingHole" H 11100 10805 50  0000 L CNN
+F 2 "MountingHole:MountingHole_3.2mm_M3_DIN965" H 11000 10850 50  0001 C CNN
+F 3 "~" H 11000 10850 50  0001 C CNN
+	1    11000 10850
+	1    0    0    -1
+$EndComp
 $EndSCHEMATC

Commit message: Revise layout
Parts:
- added C12, C13, C14: 100n, Capacitor_SMD:C_0603_1608Metric_Pad1.05x0.95mm_HandSolder, symbol Device:C
- J27: footprint Connector_JST:JST_XH_B7B-XH-A_1x07_P2.50mm_Vertical -> Connector_JST:JST_XH_B8B-XH-A_1x08_P2.50mm_Vertical; symbol Connector_Generic:Conn_01x07 -> Connector_Generic:Conn_01x08
- Y1: footprint Crystal:Crystal_SMD_5032-2Pin_5.0x3.2mm_HandSoldering -> Crystal:Crystal_SMD_5032-2Pin_5.0x3.2mm
Connections:
- net +3V3: now also C12.1, C13.1, C14.1
- net 3V3_RF: now also J27.3 (Pin_3)
- net CSN: now also J27.4 (Pin_4); no longer J27.3 (Pin_3)
- net GND: now also C12.2, C13.2, C14.2
- net IRQ: now also J27.8 (Pin_8); no longer J27.5 (Pin_5)
- net MISO: now also J27.7 (Pin_7); no longer J27.6 (Pin_6)
- net MOSI: now also J27.6 (Pin_6); no longer J27.4 (Pin_4)
- net SCK: now also J27.5 (Pin_5); no longer J27.7 (Pin_7)
Changed lines of the file:
@@
 Battery level\nsensing
 $Comp
-L Connector_Generic:Conn_01x07 J27
+L Connector_Generic:Conn_01x08 J27
 U 1 1 5E7A987D
 P 14100 2050
-F 0 "J27" H 14018 1525 50  0000 C CNN
-F 1 "NRF24 connector" H 14018 1616 50  0000 C CNN
-F 2 "Connector_JST:JST_XH_B7B-XH-A_1x07_P2.50mm_Vertical" H 14100 2050 50  0001 C CNN
+F 0 "J27" H 14100 1350 50  0000 C CNN
+F 1 "NRF24 connector" H 14100 1450 50  0000 C CNN
+F 2 "Connector_JST:JST_XH_B8B-XH-A_1x08_P2.50mm_Vertical" H 14100 2050 50  0001 C CNN
 F 3 "~" H 14100 2050 50  0001 C CNN
 	1    14100 2050
@@
 	13600 2250 13900 2250
 Wire Wire Line
-	13900 2150 13000 2150
-Wire Wire Line
 	13000 2050 13900 2050
 Wire Wire Line
 	13000 1950 13900 1950
-Text Label 13000 2150 0    50   ~ 0
+Text Label 13000 2050 0    50   ~ 0
 CSN
+Text Label 13000 1950 0    50   ~ 0
+SCK
+Text Label 13000 1850 0    50   ~ 0
+MOSI
 Text Label 13000 1750 0    50   ~ 0
-SCK
-Text Label 13000 2050 0    50   ~ 0
-MOSI
-Text Label 13000 1850 0    50   ~ 0
 MISO
-Text Label 13000 1950 0    50   ~ 0
+Text Label 13000 1650 0    50   ~ 0
 IRQ
 $Comp
@@
 	12150 1300 12600 1300
 Wire Wire Line
-	13600 1300 13600 2250
+	13600 1300 13600 2150
 Wire Wire Line
 	13600 2350 13900 2350
@@
 F 0 "Y1" V 4904 4031 50  0000 L CNN
 F 1 "8MHz" V 4995 4031 50  0000 L CNN
-F 2 "Crystal:Crystal_SMD_5032-2Pin_5.0x3.2mm_HandSoldering" H 4950 3900 50  0001 C CNN
+F 2 "Crystal:Crystal_SMD_5032-2Pin_5.0x3.2mm" H 4950 3900 50  0001 C CNN
 F 3 "~" H 4950 3900 50  0001 C CNN
 	1    4950 3900
@@
 	13600 2350 13600 3000
 Wire Wire Line
-	13000 1750 13900 1750
+	13000 1650 13900 1650
 Wire Wire Line
 	13000 1850 13900 1850
@@
 	1    0    0    -1
 $EndComp
+Wire Wire Line
+	13000 1750 13900 1750
+Wire Wire Line
+	13600 2150 13900 2150
+Connection ~ 13600 2150
+Wire Wire Line
+	13600 2150 13600 2250
+$Comp
+L Device:C C12
+U 1 1 5E3856D9
+P 9650 1750
+F 0 "C12" H 9765 1796 50  0000 L CNN
+F 1 "100n" H 9765 1705 50  0000 L CNN
+F 2 "Capacitor_SMD:C_0603_1608Metric_Pad1.05x0.95mm_HandSolder" H 9688 1600 50  0001 C CNN
+F 3 "~" H 9650 1750 50  0001 C CNN
+	1    9650 1750
+	1    0    0    -1
+$EndComp
+Wire Wire Line
+	9200 1500 9650 1500
+Wire Wire Line
+	9650 1500 9650 1600
+Connection ~ 9200 1500
+$Comp
+L power:GND #PWR030
+U 1 1 5E39BCE9
+P 9650 2100
+F 0 "#PWR030" H 9650 1850 50  0001 C CNN
+F 1 "GND" H 9655 1927 50  0000 C CNN
+F 2 "" H 9650 2100 50  0001 C CNN
+F 3 "" H 9650 2100 50  0001 C CNN
+	1    9650 2100
+	1    0    0    -1
+$EndComp
+Wire Wire Line
+	9650 1900 9650 2100
+$Comp
+L Device:C C13
+U 1 1 5E3B27F1
+P 10100 1750
+F 0 "C13" H 10215 1796 50  0000 L CNN
+F 1 "100n" H 10215 1705 50  0000 L CNN
+F 2 "Capacitor_SMD:C_0603_1608Metric_Pad1.05x0.95mm_HandSolder" H 10138 1600 50  0001 C CNN
+F 3 "~" H 10100 1750 50  0001 C CNN
+	1    10100 1750
+	1    0    0    -1
+$EndComp
+Wire Wire Line
+	9650 1500 10100 1500
+Wire Wire Line
+	10100 1500 10100 1600
+Connection ~ 9650 1500
+$Comp
+L power:GND #PWR041
+U 1 1 5E3C9708
+P 10100 2100
+F 0 "#PWR041" H 10100 1850 50  0001 C CNN
+F 1 "GND" H 10105 1927 50  0000 C CNN
+F 2 "" H 10100 2100 50  0001 C CNN
+F 3 "" H 10100 2100 50  0001 C CNN
+	1    10100 2100
+	1    0    0    -1
+$EndComp
+Wire Wire Line
+	10100 1900 10100 2100
+$Comp
+L Device:C C14
+U 1 1 5E4B0829
+P 10550 1750
+F 0 "C14" H 10665 1796 50  0000 L CNN
+F 1 "100n" H 10665 1705 50  0000 L CNN
+F 2 "Capacitor_SMD:C_0603_1608Metric_Pad1.05x0.95mm_HandSolder" H 10588 1600 50  0001 C CNN
+F 3 "~" H 10550 1750 50  0001 C CNN
+	1    10550 1750
+	1    0    0    -1
+$EndComp
+Wire Wire Line
+	10100 1500 10550 1500
+Wire Wire Line
+	10550 1500 10550 1600
+Connection ~ 10100 1500
+$Comp
+L power:GND #PWR042
+U 1 1 5E4CB16A
+P 10550 2100
+F 0 "#PWR042" H 10550 1850 50  0001 C CNN
+F 1 "GND" H 10555 1927 50  0000 C CNN
+F 2 "" H 10550 2100 50  0001 C CNN
+F 3 "" H 10550 2100 50  0001 C CNN
+	1    10550 2100
+	1    0    0    -1
+$EndComp
+Wire Wire Line
+	10550 1900 10550 2100
 $EndSCHEMATC

Commit message: Make combined PCB
Parts:
- added H4, H5, H6, H7, H8: MountingHole, MountingHole:MountingHole_3.2mm_M3_DIN965, symbol Mechanical:MountingHole
Other:
- moved on the sheet: H1, H2, H3
Changed lines of the file:
@@
 L Mechanical:MountingHole H1
 U 1 1 5E38CF71
-P 11000 10350
-F 0 "H1" H 11100 10396 50  0000 L CNN
-F 1 "MountingHole" H 11100 10305 50  0000 L CNN
-F 2 "MountingHole:MountingHole_3.2mm_M3_DIN965" H 11000 10350 50  0001 C CNN
-F 3 "~" H 11000 10350 50  0001 C CNN
-	1    11000 10350
+P 8500 10350
+F 0 "H1" H 8600 10396 50  0000 L CNN
+F 1 "MountingHole" H 8600 10305 50  0000 L CNN
+F 2 "MountingHole:MountingHole_3.2mm_M3_DIN965" H 8500 10350 50  0001 C CNN
+F 3 "~" H 8500 10350 50  0001 C CNN
+	1    8500 10350
 	1    0    0    -1
 $EndComp
@@
 L Mechanical:MountingHole H2
 U 1 1 5E38F132
-P 11000 10600
-F 0 "H2" H 11100 10646 50  0000 L CNN
-F 1 "MountingHole" H 11100 10555 50  0000 L CNN
-F 2 "MountingHole:MountingHole_3.2mm_M3_DIN965" H 11000 10600 50  0001 C CNN
-F 3 "~" H 11000 10600 50  0001 C CNN
-	1    11000 10600
+P 8500 10600
+F 0 "H2" H 8600 10646 50  0000 L CNN
+F 1 "MountingHole" H 8600 10555 50  0000 L CNN
+F 2 "MountingHole:MountingHole_3.2mm_M3_DIN965" H 8500 10600 50  0001 C CNN
+F 3 "~" H 8500 10600 50  0001 C CNN
+	1    8500 10600
 	1    0    0    -1
 $EndComp
@@
 L Mechanical:MountingHole H3
 U 1 1 5E292C58
-P 11000 10850
-F 0 "H3" H 11100 10896 50  0000 L CNN
-F 1 "MountingHole" H 11100 10805 50  0000 L CNN
-F 2 "MountingHole:MountingHole_3.2mm_M3_DIN965" H 11000 10850 50  0001 C CNN
-F 3 "~" H 11000 10850 50  0001 C CNN
-	1    11000 10850
+P 8500 10850
+F 0 "H3" H 8600 10896 50  0000 L CNN
+F 1 "MountingHole" H 8600 10805 50  0000 L CNN
+F 2 "MountingHole:MountingHole_3.2mm_M3_DIN965" H 8500 10850 50  0001 C CNN
+F 3 "~" H 8500 10850 50  0001 C CNN
+	1    8500 10850
 	1    0    0    -1
 $EndComp
@@
 Wire Wire Line
 	10550 1900 10550 2100
+$Comp
+L Mechanical:MountingHole H4
+U 1 1 5E321FB8
+P 9500 10350
+F 0 "H4" H 9600 10396 50  0000 L CNN
+F 1 "MountingHole" H 9600 10305 50  0000 L CNN
+F 2 "MountingHole:MountingHole_3.2mm_M3_DIN965" H 9500 10350 50  0001 C CNN
+F 3 "~" H 9500 10350 50  0001 C CNN
+	1    9500 10350
+	1    0    0    -1
+$EndComp
+$Comp
+L Mechanical:MountingHole H5
+U 1 1 5E321FC2
+P 9500 10600
+F 0 "H5" H 9600 10646 50  0000 L CNN
+F 1 "MountingHole" H 9600 10555 50  0000 L CNN
+F 2 "MountingHole:MountingHole_3.2mm_M3_DIN965" H 9500 10600 50  0001 C CNN
+F 3 "~" H 9500 10600 50  0001 C CNN
+	1    9500 10600
+	1    0    0    -1
+$EndComp
+$Comp
+L Mechanical:MountingHole H6
+U 1 1 5E321FCC
+P 9500 10850
+F 0 "H6" H 9600 10896 50  0000 L CNN
+F 1 "MountingHole" H 9600 10805 50  0000 L CNN
+F 2 "MountingHole:MountingHole_3.2mm_M3_DIN965" H 9500 10850 50  0001 C CNN
+F 3 "~" H 9500 10850 50  0001 C CNN
+	1    9500 10850
+	1    0    0    -1
+$EndComp
+$Comp
+L Mechanical:MountingHole H7
+U 1 1 5E33A1E2
+P 10400 10350
+F 0 "H7" H 10500 10396 50  0000 L CNN
+F 1 "MountingHole" H 10500 10305 50  0000 L CNN
+F 2 "MountingHole:MountingHole_3.2mm_M3_DIN965" H 10400 10350 50  0001 C CNN
+F 3 "~" H 10400 10350 50  0001 C CNN
+	1    10400 10350
+	1    0    0    -1
+$EndComp
+$Comp
+L Mechanical:MountingHole H8
+U 1 1 5E393426
+P 10400 10600
+F 0 "H8" H 10500 10646 50  0000 L CNN
+F 1 "MountingHole" H 10500 10555 50  0000 L CNN
+F 2 "MountingHole:MountingHole_3.2mm_M3_DIN965" H 10400 10600 50  0001 C CNN
+F 3 "~" H 10400 10600 50  0001 C CNN
+	1    10400 10600
+	1    0    0    -1
+$EndComp
 $EndSCHEMATC

Commit message: Finalize layout
Parts:
- added H10, H9: MountingHole, MountingHole:MountingHole_3.2mm_M3_DIN965, symbol Mechanical:MountingHole
- H4, H5, H6, H7, H8: footprint MountingHole:MountingHole_3.2mm_M3_DIN965 -> MountingHole:MountingHole_2.7mm_M2.5_DIN965
Changed lines of the file:
@@
 F 0 "H4" H 9600 10396 50  0000 L CNN
 F 1 "MountingHole" H 9600 10305 50  0000 L CNN
-F 2 "MountingHole:MountingHole_3.2mm_M3_DIN965" H 9500 10350 50  0001 C CNN
+F 2 "MountingHole:MountingHole_2.7mm_M2.5_DIN965" H 9500 10350 50  0001 C CNN
 F 3 "~" H 9500 10350 50  0001 C CNN
 	1    9500 10350
@@
 F 0 "H5" H 9600 10646 50  0000 L CNN
 F 1 "MountingHole" H 9600 10555 50  0000 L CNN
-F 2 "MountingHole:MountingHole_3.2mm_M3_DIN965" H 9500 10600 50  0001 C CNN
+F 2 "MountingHole:MountingHole_2.7mm_M2.5_DIN965" H 9500 10600 50  0001 C CNN
 F 3 "~" H 9500 10600 50  0001 C CNN
 	1    9500 10600
@@
 F 0 "H6" H 9600 10896 50  0000 L CNN
 F 1 "MountingHole" H 9600 10805 50  0000 L CNN
-F 2 "MountingHole:MountingHole_3.2mm_M3_DIN965" H 9500 10850 50  0001 C CNN
+F 2 "MountingHole:MountingHole_2.7mm_M2.5_DIN965" H 9500 10850 50  0001 C CNN
 F 3 "~" H 9500 10850 50  0001 C CNN
 	1    9500 10850
@@
 F 0 "H7" H 10500 10396 50  0000 L CNN
 F 1 "MountingHole" H 10500 10305 50  0000 L CNN
-F 2 "MountingHole:MountingHole_3.2mm_M3_DIN965" H 10400 10350 50  0001 C CNN
+F 2 "MountingHole:MountingHole_2.7mm_M2.5_DIN965" H 10400 10350 50  0001 C CNN
 F 3 "~" H 10400 10350 50  0001 C CNN
 	1    10400 10350
@@
 F 0 "H8" H 10500 10646 50  0000 L CNN
 F 1 "MountingHole" H 10500 10555 50  0000 L CNN
-F 2 "MountingHole:MountingHole_3.2mm_M3_DIN965" H 10400 10600 50  0001 C CNN
+F 2 "MountingHole:MountingHole_2.7mm_M2.5_DIN965" H 10400 10600 50  0001 C CNN
 F 3 "~" H 10400 10600 50  0001 C CNN
 	1    10400 10600
 	1    0    0    -1
 $EndComp
+$Comp
+L Mechanical:MountingHole H9
+U 1 1 5E301527
+P 10400 10850
+F 0 "H9" H 10500 10896 50  0000 L CNN
+F 1 "MountingHole" H 10500 10805 50  0000 L CNN
+F 2 "MountingHole:MountingHole_3.2mm_M3_DIN965" H 10400 10850 50  0001 C CNN
+F 3 "~" H 10400 10850 50  0001 C CNN
+	1    10400 10850
+	1    0    0    -1
+$EndComp
+$Comp
+L Mechanical:MountingHole H10
+U 1 1 5E302819
+P 11150 10350
+F 0 "H10" H 11250 10396 50  0000 L CNN
+F 1 "MountingHole" H 11250 10305 50  0000 L CNN
+F 2 "MountingHole:MountingHole_3.2mm_M3_DIN965" H 11150 10350 50  0001 C CNN
+F 3 "~" H 11150 10350 50  0001 C CNN
+	1    11150 10350
+	1    0    0    -1
+$EndComp
